File: projects/reflex-machine/reflex-machine.kicad_sch (KiCad schematic)
At the start: 123 parts, among them J1 12V_IN, J10 MAG9, J11 MAG10, J12 COIN, J13 BUTTONS, J14 STATUS_LEDS, J15 7SEG, J16 MEGA SPARE, J17 ESP32 SPARE, J2 MAG1, J3 MAG2, J4 MAG3, J5 MAG4, J6 MAG5, J7 MAG6, J8 MAG7, J9 MAG8, Q1 IRLZ44N, Q10 IRLZ44N, Q2 IRLZ44N, Q3 IRLZ44N, Q4 IRLZ44N, Q5 IRLZ44N, Q6 IRLZ44N, Q7 IRLZ44N, Q8 IRLZ44N, Q9 IRLZ44N, U1 5V 2A module (K7805-2000R3), U2 PC817, U3 74HC595N

Commit message: fix(MD-T8): place decoupling caps at their IC supply pins (blinky C3, reflex C13)
Co-Authored-By: Claude Opus 5.5 <noreply@anthropic.com>
Other:
- title: Reflex Machine Controller Shield -> reflex-machine

Commit message: feat(P1-T9b): fixtures on the parts registry (pins by function, strict mode)
Co-Authored-By: Claude Opus 5.5 <noreply@anthropic.com>
Parts:
- C1: LCSC C48935382 -> (none)
- C2, C6: symbol Device:C -> Device:C_Polarized; LCSC C47344177 -> (none)
- C8: LCSC C49002957 -> (none)
- D1: LCSC C294003 -> (none)
- D11, D12, D13, D14, D15, D16, D17, D18, D19, D20: LCSC C2476 -> (none)
- D2: LCSC C2985028 -> (none)
- D21, D22, D23, D24, D25, D26, D27, D28, D29, D30: LCSC C2895470 -> (none)
- R21, R22, R23, R24, R25, R26, R27, R28, R29, R30, R42, R47, R48, R49, R50: LCSC C2649453 -> (none)

Commit message: fix(P1-T9b): keep LCSC ids, package family match, PR-BYNAME
Co-Authored-By: Claude Opus 5.5 <noreply@anthropic.com>
Parts:
- C1: LCSC (none) -> C48935382
- C2, C6: LCSC (none) -> C47344177
- C8: LCSC (none) -> C49002957
- D1: LCSC (none) -> C294003
- D11, D12, D13, D14, D15, D16, D17, D18, D19, D20: LCSC (none) -> C2476
- D2: LCSC (none) -> C2985028
- D21, D22, D23, D24, D25, D26, D27, D28, D29, D30: LCSC (none) -> C2895470
- R21, R22, R23, R24, R25, R26, R27, R28, R29, R30, R42, R47, R48, R49, R50: LCSC (none) -> C2649453
