File: projects/uno-toggle/uno-toggle.kicad_sch (KiCad schematic)
At the start: 9 parts, among them SW1 BTN1, SW2 BTN2

Commit message: feat(P1-T9b): fixtures on the parts registry (pins by function, strict mode)
Co-Authored-By: Claude Opus 5.5 <noreply@anthropic.com>
Parts:
- D1: LCSC C2895470 -> (none)
Changed lines of the file:
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@@
-			)
-		)
-		(property "LCSC" "C2895470"
-			(at 50.8 195.58 0)
-			(show_name no)
-			(do_not_autoplace no)
-			(hide yes)
-			(effects
-				(font
-					(size 1.27 1.27)
-				)
 			)
 		)

Commit message: fix(P1-T9b): keep LCSC ids, package family match, PR-BYNAME
Co-Authored-By: Claude Opus 5.5 <noreply@anthropic.com>
Parts:
- D1: LCSC (none) -> C2895470
Changed lines of the file:
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@@
+			)
+		)
+		(property "LCSC" "C2895470"
+			(at 50.8 195.58 0)
+			(show_name no)
+			(do_not_autoplace no)
+			(hide yes)
+			(effects
+				(font
+					(size 1.27 1.27)
+				)
 			)
 		)
